File: PORTABLE_ECG_MACHINE/PORTABLE_ECG_MACHINE.kicad_sch (KiCad schematic)
At the start: 87 parts, among them IC1 AD8232ACPZ, J1 UART, J2 AudioJack3, J3 Li-Ion 3.7 CONN, J4 USB_C_Receptacle_USB2.0, J5 Conn_01x06_Male, Q1 BSS138, Q2 BSS138, SW1 SW_SPDT, U1 SSD1306, U2 CP2102-GM, U3 ATmega328PB-A, U4 TC1262-33, U5 TP4056, Y1 16MHZ

Commit message: version 2.0 | oled 128*64
new version created substituted 128*64 instead of 128*64. EESCHEMA and PCBNEW completed. OLED 128*64 3D MODEL need to fix
Parts:
- removed C8, C9: 1uf, Capacitor_SMD:C_0603_1608Metric, symbol Adafruit OLED 128x32 Mono I2C-eagle-import:CAP_CERAMIC0402
- removed U1: SSD1306, SSD1306:SSD1306, symbol SSD1306:SSD1306
- added U6: SSD1306, Display:OLED-128O064D, symbol user_symbol:SSD1306
- C6: value 10uf -> 2.2UF
- C7: value 10uf -> 10UF
- R4: value 330k -> 390K
Connections:
- net 3.3V: now also R6.1, U6.11 (BS1), U6.6 (VBAT), U6.9 (VDD); no longer R6.2
- net GND: now also C6.2 (P$2), C7.2 (P$2), U6.1 (NC), U6.10 (BS0), U6.12 (BS2), U6.13 (/CS), U6.29 (VLSS), U6.30 (NC), U6.8 (VSS); no longer C5.1 (P$1), C6.1 (P$1), C7.1 (P$1)
- net SCL_3.3: now also U6.18 (D0/SPI_SCLK/I2C_SCK)
- net SDA_3.3: now also R6.2, U6.19 (D1/SPI_SDIN/I2C_SDA), U6.20 (D2/I2C_SDA); no longer R6.1
- net at C4.1 (P$1): now also U6.3 (C2N)
- net at R4.1: now also U6.26 (IREF)
- net at C4.2 (P$2): now also U6.2 (C2P)
- net at C5.2 (P$2): now also U6.5 (C1N)
- new net: C7.1 (P$1), U6.28 (VCC)
- new net: C5.1 (P$1), U6.4 (C1P)
- new net: C6.1 (P$1), U6.27 (VCOMH)
- no-connect marks 16 -> 21
Other:
- note added: "5V TO 3.3V LOGIC LEVEL CONVERTER"
- note added: "OLED 128*64"
- note removed: "OLED 128*32"
- note removed: "OPTIONAL 5V TO 3.3V LOGIC LEVEL CONVERTER"
- company: (none) -> GROUP 5
- title: (none) -> P-ECG
- moved on the sheet: B_TEMP1, C12, C13, C14, C20, C21, C22, C23, C24, D+1, D-1, D1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
